File: mcprog.brd (EAGLE design)
At the start: 45.8 x 37.2 mm, 52 parts, among them IC1 MCP2210SO, IC2 MCP1703SOT-89, J1 AVRSPI-61.27, J2 AVRSPI-62.56-V, Q1 MOSFET-NCHANNELSMD, X1 MICRO-USB-AB, X2 12MHz

Commit message: attach PROG led to GPIO6 instead of GPIO8 GPIO8 refused to be an output for some unknown reason
Connections:
- removed net N$30: IC1.16, R25.1
- new net N$16: IC1.14, R25.1
Routing:
- net N$30: track 19.8 -> 0.00 mm, vias 2 -> 0
- net N$16: track 0.00 -> 17.1 mm, vias 0 -> 2
Other:
- board text added: "v1.1"
- board text removed: "v1.0"
Changed lines of the file:
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@@
 <?xml version="1.0" encoding="utf-8"?>
 <!DOCTYPE eagle SYSTEM "eagle.dtd">
-<eagle version="6.5.0">
+<eagle version="6.6.0">
 <drawing>
 <settings>
@@
 <text x="26.8" y="29.8" size="1" layer="29" font="vector" ratio="16" rot="R90">ERROR</text>
 <text x="30.4" y="28.4" size="1" layer="29" font="vector" ratio="16" rot="R90">V_TARGET</text>
-<text x="2.6" y="3" size="1" layer="29" font="vector" ratio="16" rot="R315" align="bottom-center">v1.0</text>
-<text x="2.6" y="3" size="1" layer="1" font="vector" ratio="16" rot="R315" align="bottom-center">v1.0</text>
+<text x="2.6" y="3" size="1" layer="29" font="vector" ratio="16" rot="R315" align="bottom-center">v1.1</text>
+<text x="2.6" y="3" size="1" layer="1" font="vector" ratio="16" rot="R315" align="bottom-center">v1.1</text>
 <text x="5.2" y="5.2" size="1" layer="16" font="vector" ratio="16" rot="SR315" align="bottom-center">www.bytewerk.org</text>
 <text x="5.2" y="5.2" size="1" layer="30" font="vector" ratio="16" rot="SR315" align="bottom-center">www.bytewerk.org</text>
 <text x="3.8" y="4.2" size="1.5" layer="16" font="vector" ratio="16" rot="SR315" align="bottom-center">mcprog</text>
 <text x="3.8" y="4.2" size="1.5" layer="30" font="vector" ratio="16" rot="SR315" align="bottom-center">mcprog</text>
-<text x="2.6" y="3" size="1" layer="16" font="vector" ratio="16" rot="R315" align="bottom-center">v1.0</text>
-<text x="2.6" y="3" size="1" layer="30" font="vector" ratio="16" rot="R315" align="bottom-center">v1.0</text>
+<text x="2.6" y="3" size="1" layer="16" font="vector" ratio="16" rot="R315" align="bottom-center">v1.1</text>
+<text x="2.6" y="3" size="1" layer="30" font="vector" ratio="16" rot="R315" align="bottom-center">v1.1</text>
 </plain>
 <attributes>
@@
 <wire x1="24.01" y1="33.72" x2="24.01" y2="32.73" width="0.2" layer="1"/>
 </signal>
-<signal name="N$30">
-<contactref element="R25" pad="1"/>
-<contactref element="IC1" pad="16"/>
-<via x="24" y="29.6" extent="1-16" drill="0.3"/>
-<wire x1="22.4" y1="28.2" x2="22.4" y2="15.6" width="0.2" layer="16"/>
-<via x="22" y="15.2" extent="1-16" drill="0.3"/>
-<wire x1="21.875" y1="15.075" x2="19.05" y2="15.075" width="0.2" layer="1"/>
-<wire x1="21.875" y1="15.075" x2="22" y2="15.2" width="0.2" layer="1"/>
-<wire x1="22.4" y1="15.6" x2="22" y2="15.2" width="0.2" layer="16"/>
-<wire x1="22.4" y1="28.2" x2="23.8" y2="29.6" width="0.2" layer="16"/>
-<wire x1="23.8" y1="29.6" x2="24" y2="29.6" width="0.2" layer="16"/>
-<wire x1="24.01" y1="31.03" x2="24" y2="31.02" width="0.2" layer="1"/>
-<wire x1="24" y1="31.02" x2="24" y2="29.6" width="0.2" layer="1"/>
-</signal>
 <signal name="N$32">
 <contactref element="LED5" pad="A"/>
@@
 <wire x1="33.95" y1="9.65" x2="34" y2="9.6" width="0.2" layer="16"/>
 </signal>
+<signal name="N$16">
+<contactref element="IC1" pad="14"/>
+<contactref element="R25" pad="1"/>
+<via x="24" y="29.6" extent="1-16" drill="0.3"/>
+<wire x1="22.4" y1="28.2" x2="22.4" y2="18.4" width="0.2" layer="16"/>
+<via x="21.8" y="17.8" extent="1-16" drill="0.3"/>
+<wire x1="22.4" y1="28.2" x2="23.8" y2="29.6" width="0.2" layer="16"/>
+<wire x1="23.8" y1="29.6" x2="24" y2="29.6" width="0.2" layer="16"/>
+<wire x1="24.01" y1="31.03" x2="24" y2="31.02" width="0.2" layer="1"/>
+<wire x1="24" y1="31.02" x2="24" y2="29.6" width="0.2" layer="1"/>
+<wire x1="22.4" y1="18.4" x2="21.8" y2="17.8" width="0.2" layer="16"/>
+<wire x1="19.05" y1="17.615" x2="21.615" y2="17.615" width="0.2" layer="1"/>
+<wire x1="21.615" y1="17.615" x2="21.8" y2="17.8" width="0.2" layer="1"/>
+</signal>
 </signals>

Commit message: v1.2 with various small changes
Parts:
- removed JUMPER1: JUMPER-2_10B, bytewerk-jumper:JMP2-1B
- removed S1: (no value), switch:255SB
- added JP1: (no value), jumper:JP2
- added JP2: (no value), jumper:JP1
- C2: value 22uF/10V -> 2u2F/10V
- C5: value 470nF/10V -> 220nF/10V
- C6, C7: value 22uF/10V -> 10uF/10V
- R21, R22: value 100R -> 22R
- moved D1 24.6 mm to (21.5, 25.3)
- moved J1 2.01 mm to (38.3, 31.8)
- moved R20 1.31 mm to (6.08, 12.0), turned to 270 degrees
- moved C9 1.14 mm to (10.2, 26.5), turned to 270 degrees
- moved C1 0.80 mm to (28.8, 7.70)
- moved C2 0.60 mm to (28.6, 5.80)
Connections:
- net +3V3: now also JP1.1; no longer S1.3
- net +5V: now also JP1.3; no longer S1.1
- net N$27: now also D1.A, JP2.1; no longer D1.C, JUMPER1.1
- net VDD: now also JP1.2, JP2.2; no longer D1.A, S1.2
- net V_TARGET: now also D1.C; no longer JUMPER1.2
Routing:
- net N$27: track 3.69 -> 20.1 mm, vias 0 -> 1
- net V_TARGET: track 62.2 -> 49.5 mm, vias 0 -> 2
- net MISO: track 45.3 -> 40.3 mm, vias 3 -> 4
- net VDD: track 91.0 -> 87.0 mm
- net N$1: track 8.83 -> 10.5 mm
- net N$2: track 6.14 -> 7.71 mm
- net GND: track 41.7 -> 43.0 mm, vias 5 -> 6
- net N$3: track 3.40 -> 4.52 mm
Other:
- board text added: "PWR TARGET"
- board text added: "TARGET"
- board text added: "USB"
- board text added: "v1.2"
- board text removed: "1->"
- board text removed: "SUPPLY V_TARGET"
- board text removed: "USB CFG"
- board text removed: "V_TARGET"
- board text removed: "v1.1"
