File: mcprog.sch (EAGLE design)
At the start: 52 parts, among them IC1 MCP2210SO, IC2 MCP1703SOT-89, J1 AVRSPI-61.27, J2 AVRSPI-62.56-V, Q1 MOSFET-NCHANNELSMD, X1 MICRO-USB-AB, X2 12MHz

Commit message: v1.2 with various small changes
Parts:
- removed JUMPER1: JUMPER-2_10B, bytewerk-jumper:JUMPER-2_10B
- removed S1: (no value), switch:255SB
- added JP1: (no value), jumper:JP2E
- added JP2: (no value), jumper:JP1E
- C2: value 22uF/10V -> 2u2F/10V
- C5: value 470nF/10V -> 220nF/10V
- C6, C7: value 22uF/10V -> 10uF/10V
- R21, R22: value 100R -> 22R
Connections:
- net +3V3: now also JP1.1; no longer S1.S
- net +5V: now also JP1.3; no longer S1.O
- net N$27: now also D1.A, JP2.1; no longer D1.C, JUMPER1.1
- net VDD: now also JP1.2, JP2.2; no longer D1.A, S1.P
- net V_TARGET: now also D1.C; no longer JUMPER1.2
Other:
- note added: "V_GS(th) << 1,5V! z.B. TSM2311"
- note removed: "Achtung: V_GS(th) << 1,5V!"
- moved on the sheet: R2
Changed lines of the file:
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@@
 <part name="LED3" library="bytewerk-led" deviceset="LED0603" device=""/>
 <part name="C1" library="bytewerk-passive" deviceset="C" device="0603" value="100nF/10V"/>
-<part name="C2" library="bytewerk-passive" deviceset="C" device="1206" value="22uF/10V"/>
+<part name="C2" library="bytewerk-passive" deviceset="C" device="1206" value="2u2F/10V"/>
 <part name="R1" library="bytewerk-passive" deviceset="R" device="0603" value="100R"/>
 <part name="R2" library="bytewerk-passive" deviceset="R" device="0603" value="100R"/>
@@
 <part name="U$11" library="bytewerk-symbol" deviceset="GND" device=""/>
 <part name="IC1" library="mcp2210" deviceset="MCP2210" device="SO"/>
-<part name="R21" library="bytewerk-passive" deviceset="R" device="0603" value="100R"/>
-<part name="R22" library="bytewerk-passive" deviceset="R" device="0603" value="100R"/>
+<part name="R21" library="bytewerk-passive" deviceset="R" device="0603" value="22R"/>
+<part name="R22" library="bytewerk-passive" deviceset="R" device="0603" value="22R"/>
 <part name="D1" library="bytewerk-passive" deviceset="1N5819HW" device=""/>
-<part name="C5" library="bytewerk-passive" deviceset="C" device="0603" value="470nF/10V"/>
+<part name="C5" library="bytewerk-passive" deviceset="C" device="0603" value="220nF/10V"/>
 <part name="R23" library="bytewerk-passive" deviceset="R" device="0603" value="10k"/>
 <part name="IC2" library="bytewerk-vreg" deviceset="MCP1703" device="SOT-89"/>
@@
 <part name="U$14" library="bytewerk-symbol" deviceset="+5V" device=""/>
 <part name="U$15" library="bytewerk-symbol" deviceset="+3V3" device=""/>
-<part name="C6" library="bytewerk-passive" deviceset="C" device="1206" value="22uF/10V"/>
-<part name="C7" library="bytewerk-passive" deviceset="C" device="1206" value="22uF/10V"/>
+<part name="C6" library="bytewerk-passive" deviceset="C" device="1206" value="10uF/10V"/>
+<part name="C7" library="bytewerk-passive" deviceset="C" device="1206" value="10uF/10V"/>
 <part name="C8" library="bytewerk-passive" deviceset="C" device="0603" value="100nF/10V"/>
 <part name="C9" library="bytewerk-passive" deviceset="C" device="0603" value="100nF/10V"/>
@@
 <part name="R26" library="bytewerk-passive" deviceset="R" device="0603" value="470R"/>
 <part name="LED5" library="bytewerk-led" deviceset="LED0603" device=""/>
-<part name="S1" library="switch" deviceset="255SB" device=""/>
 <part name="U$4" library="bytewerk-symbol" deviceset="+5V" device=""/>
 <part name="U$12" library="bytewerk-symbol" deviceset="+3V3" device=""/>
@@
 <part name="U$18" library="bytewerk-symbol" deviceset="+3V3" device=""/>
 <part name="U$19" library="bytewerk-symbol" deviceset="GND" device=""/>
-<part name="JUMPER1" library="bytewerk-jumper" deviceset="JUMPER-2" device="_10B"/>
 <part name="R11" library="bytewerk-passive" deviceset="R" device="0603" value="0R"/>
 <part name="U$20" library="bytewerk-symbol" deviceset="GND" device=""/>
@@
 <part name="U$16" library="bytewerk-symbol" deviceset="GND" device=""/>
 <part name="Q1" library="bytewerk-transistor" deviceset="MOSFET-NCHANNEL" device="SMD"/>
+<part name="JP1" library="jumper" deviceset="JP2E" device=""/>
+<part name="JP2" library="jumper" deviceset="JP1E" device=""/>
 </parts>
 <sheets>
 <sheet>
 <plain>
-<text x="66.04" y="43.18" size="1.778" layer="98">Achtung: V_GS(th) &lt;&lt; 1,5V!</text>
+<text x="63.5" y="43.18" size="1.778" layer="98">V_GS(th) &lt;&lt; 1,5V!
+z.B. TSM2311</text>
 </plain>
 <instances>
@@
 <instance part="C2" gate="G$1" x="78.74" y="86.36" rot="R90"/>
 <instance part="R1" gate="G$1" x="162.56" y="88.9"/>
-<instance part="R2" gate="G$1" x="160.02" y="86.36"/>
+<instance part="R2" gate="G$1" x="157.48" y="86.36"/>
 <instance part="R3" gate="G$1" x="162.56" y="83.82"/>
 <instance part="R4" gate="G$1" x="162.56" y="71.12"/>
@@
 <instance part="R21" gate="G$1" x="45.72" y="147.32"/>
 <instance part="R22" gate="G$1" x="40.64" y="144.78"/>
-<instance part="D1" gate="G$1" x="251.46" y="96.52" rot="R270"/>
+<instance part="D1" gate="G$1" x="251.46" y="86.36" rot="R270"/>
 <instance part="C5" gate="G$1" x="55.88" y="86.36" rot="R90"/>
 <instance part="R23" gate="G$1" x="58.42" y="104.14" rot="R270"/>
@@
 <instance part="R26" gate="G$1" x="195.58" y="132.08" rot="R270"/>
 <instance part="LED5" gate="G$1" x="195.58" y="121.92" rot="R270"/>
-<instance part="S1" gate="1" x="101.6" y="76.2" rot="R270"/>
-<instance part="U$4" gate="G$1" x="114.3" y="81.28"/>
-<instance part="U$12" gate="G$1" x="119.38" y="78.74"/>
+<instance part="U$4" gate="G$1" x="106.68" y="48.26"/>
+<instance part="U$12" gate="G$1" x="111.76" y="45.72"/>
 <instance part="Q2" gate="G$1" x="33.02" y="40.64" rot="R180"/>
 <instance part="R28" gate="G$1" x="40.64" y="48.26" rot="R180"/>
 <instance part="U$18" gate="G$1" x="33.02" y="53.34"/>
 <instance part="U$19" gate="G$1" x="55.88" y="73.66"/>
-<instance part="JUMPER1" gate="G$1" x="251.46" y="88.9" rot="R90"/>
 <instance part="R11" gate="G$1" x="40.64" y="149.86"/>
 <instance part="U$20" gate="G$1" x="251.46" y="50.8"/>
@@
 <instance part="U$16" gate="G$1" x="71.12" y="12.7"/>
 <instance part="Q1" gate="G$1" x="58.42" y="33.02" rot="MR0"/>
+<instance part="JP1" gate="1" x="109.22" y="27.94" rot="R180"/>
+<instance part="JP2" gate="A" x="246.38" y="96.52" rot="R90"/>
 </instances>
 <busses>
@@
 <segment>
 <pinref part="J1" gate="G$1" pin="SCK"/>
-<wire x1="175.26" y1="86.36" x2="165.1" y2="86.36" width="0.1524" layer="91"/>
+<wire x1="175.26" y1="86.36" x2="162.56" y2="86.36" width="0.1524" layer="91"/>
 <pinref part="R2" gate="G$1" pin="2"/>
 </segment>
@@
 </segment>
 <segment>
-<pinref part="S1" gate="1" pin="O"/>
-<wire x1="106.68" y1="76.2" x2="114.3" y2="76.2" width="0.1524" layer="91"/>
 <pinref part="U$4" gate="G$1" pin="+5V"/>
-<wire x1="114.3" y1="76.2" x2="114.3" y2="78.74" width="0.1524" layer="91"/>
+<pinref part="JP1" gate="1" pin="3"/>
+<wire x1="106.68" y1="45.72" x2="106.68" y2="30.48" width="0.1524" layer="91"/>
 </segment>
 <segment>
@@
 <segment>
 <pinref part="R2" gate="G$1" pin="1"/>
-<wire x1="154.94" y1="86.36" x2="132.08" y2="86.36" width="0.1524" layer="91"/>
+<wire x1="152.4" y1="86.36" x2="132.08" y2="86.36" width="0.1524" layer="91"/>
 <label x="134.62" y="86.36" size="1.778" layer="95"/>
 </segment>
@@
 </segment>
 <segment>
-<pinref part="S1" gate="1" pin="S"/>
-<wire x1="106.68" y1="71.12" x2="119.38" y2="71.12" width="0.1524" layer="91"/>
 <pinref part="U$12" gate="G$1" pin="+3V3"/>
-<wire x1="119.38" y1="71.12" x2="119.38" y2="78.74" width="0.1524" layer="91"/>
+<wire x1="111.76" y1="30.48" x2="111.76" y2="45.72" width="0.1524" layer="91"/>
+<pinref part="JP1" gate="1" pin="1"/>
 </segment>
 <segment>
@@
 </segment>
 <segment>
-<wire x1="251.46" y1="111.76" x2="251.46" y2="101.6" width="0.1524" layer="91"/>
+<wire x1="251.46" y1="111.76" x2="251.46" y2="99.06" width="0.1524" layer="91"/>
 <label x="251.46" y="104.14" size="1.778" layer="95" rot="R90"/>
-<pinref part="D1" gate="G$1" pin="A"/>
-</segment>
-<segment>
-<pinref part="S1" gate="1" pin="P"/>
-<wire x1="96.52" y1="73.66" x2="88.9" y2="73.66" width="0.1524" layer="91"/>
-<label x="88.9" y="73.66" size="1.778" layer="95"/>
+<pinref part="JP2" gate="A" pin="2"/>
+<wire x1="248.92" y1="99.06" x2="251.46" y2="99.06" width="0.1524" layer="91"/>
 </segment>
 <segment>
@@
 <pinref part="Q3" gate="G$1" pin="G"/>
 <wire x1="86.36" y1="40.64" x2="78.74" y2="40.64" width="0.1524" layer="91"/>
-<wire x1="86.36" y1="40.64" x2="96.52" y2="40.64" width="0.1524" layer="91"/>
+<wire x1="86.36" y1="40.64" x2="109.22" y2="40.64" width="0.1524" layer="91"/>
 <junction x="86.36" y="40.64"/>
 <label x="91.44" y="40.64" size="1.778" layer="95"/>
+<pinref part="JP1" gate="1" pin="2"/>
+<wire x1="109.22" y1="40.64" x2="109.22" y2="30.48" width="0.1524" layer="91"/>
 </segment>
 <segment>
@@
 </segment>
 </net>
-<net name="N$27" class="0">
-<segment>
-<pinref part="JUMPER1" gate="G$1" pin="1"/>
-<pinref part="D1" gate="G$1" pin="C"/>
-<wire x1="251.46" y1="91.44" x2="251.46" y2="93.98" width="0.1524" layer="91"/>
-</segment>
-</net>
 <net name="V_TARGET" class="0">
 <segment>
-<pinref part="JUMPER1" gate="G$1" pin="2"/>
-<wire x1="251.46" y1="86.36" x2="251.46" y2="78.74" width="0.1524" layer="91"/>
 <wire x1="251.46" y1="78.74" x2="233.68" y2="78.74" width="0.1524" layer="91"/>
 <label x="236.22" y="78.74" size="1.778" layer="95"/>
@@
 <pinref part="R18" gate="G$1" pin="1"/>
 <wire x1="251.46" y1="76.2" x2="251.46" y2="78.74" width="0.1524" layer="91"/>
+<pinref part="D1" gate="G$1" pin="C"/>
+<wire x1="251.46" y1="83.82" x2="251.46" y2="78.74" width="0.1524" layer="91"/>
 <junction x="251.46" y="78.74"/>
 </segment>
@@
 </segment>
 </net>
+<net name="N$27" class="0">
+<segment>
+<pinref part="JP2" gate="A" pin="1"/>
+<wire x1="251.46" y1="96.52" x2="248.92" y2="96.52" width="0.1524" layer="91"/>
+<pinref part="D1" gate="G$1" pin="A"/>
+<wire x1="251.46" y1="96.52" x2="251.46" y2="91.44" width="0.1524" layer="91"/>
+</segment>
+</net>
 </nets>
 </sheet>
@@
 </schematic>
 </drawing>
+<compatibility>
+<note version="6.3" minversion="6.2.2" severity="warning">
+Since Version 6.2.2 text objects can contain more than one line,
+which will not be processed correctly with this version.
+</note>
+</compatibility>
 </eagle>
